File: kicad/guitar_preamp.kicad_pcb (KiCad board)
At the start: 2 copper layers, 70 x 50 mm, 32 parts, among them J1 IN (from PASSIVE jack NC lug), J2 BAT+ (TP4056 OUT+), J3 ACTIVE jack Tip/Sleeve, U1 MCP6022

Commit message: v3 ПРЕДУСИЛИТЕЛЬ ДЛЯ ГИТАРЫ v3: буфер + 2-полосный темброблок, 1S Li-ion, громкость B500K push-pull (актив/пассив), светодиод питания
Parts:
- removed RV1: A25k VOLUME, Connector_Wire:SolderWire-0.5sqmm_1x03_P4.6mm_D0.9mm_OD2.1mm
- added J7: LED (A / K), Connector_Wire:SolderWire-0.5sqmm_1x02_P4.6mm_D0.9mm_OD2.1mm, F.Cu at (167.0, 108.0)
- added R13: 100k, Resistor_THT:R_Axial_DIN0207_L6.3mm_D2.5mm_P7.62mm_Horizontal, F.Cu at (164.5, 124.0)
- added R15: 4.7k, Resistor_THT:R_Axial_DIN0207_L6.3mm_D2.5mm_P7.62mm_Horizontal, F.Cu at (153.0, 108.8)
- C1: value 100p -> 47p
- J1: value IN (from PASSIVE jack NC lug) -> IN (от SW1B, экранир. провод)
- J3: value ACTIVE jack Tip/Sleeve -> OUT (к SW1A) / GND
- U1: value MCP6022 -> MCP6022/OPA2316
- moved J2 2.69 mm to (163.5, 103.0)
- moved R10 2.69 mm to (159.0, 103.0)
- moved C9 2.20 mm to (152.0, 114.2)
- moved J3 2.00 mm to (166.0, 128.0)
Connections:
- R9 pad 1: VOLW -> N4
Routing:
- net GND: track 107.7 -> 127.6 mm
- net LEDA: track 0.00 -> 6.71 mm
- net VOLW: track 6.08 -> 0.00 mm
- net N4: track 11.5 -> 6.58 mm
- net VCC: track 31.9 -> 36.7 mm
- net OUT: track 7.51 -> 9.51 mm
- net OUTB: track 50.8 -> 49.2 mm
- net VREF: track 55.1 -> 54.3 mm
Other:
- board text added: "GTR PRE v3"
- board text added: "GUITAR PRE v3 1S Li-ion"
- board text added: "LED+"
- board text added: "LED-"
- board text removed: "GTR PRE v1.0"
- board text removed: "GUITAR PRE v1.0 MCP6022 1S"
- board text removed: "V1"
- board text removed: "V2"
- board text removed: "V3"
