File: kicad/guitar_preamp.kicad_sch (KiCad schematic)
At the start: 32 parts, among them J1 IN (from PASSIVE jack NC lug), J2 BAT+ (TP4056 OUT+), J3 ACTIVE jack Tip/Sleeve, U1 MCP6022

Commit message: v3 ПРЕДУСИЛИТЕЛЬ ДЛЯ ГИТАРЫ v3: буфер + 2-полосный темброблок, 1S Li-ion, громкость B500K push-pull (актив/пассив), светодиод питания
Parts:
- added C13: 1n, symbol Device:C
- added D1: LED красн. 3мм, symbol Device:LED
- added J4: Выход 6.3 стерео TRS, symbol Connector_Audio:AudioJack3
- added J5: Звукосниматели: COM/GND, symbol Connector_Generic:Conn_01x02
- added J6: TP4056 OUT+/OUT-, symbol Connector_Generic:Conn_01x02
- added J7: LED (A / K), Connector_Wire:SolderWire-0.5sqmm_1x02_P4.6mm_D0.9mm_OD2.1mm, symbol Connector_Generic:Conn_01x02
- added R13: 100k, Resistor_THT:R_Axial_DIN0207_L6.3mm_D2.5mm_P7.62mm_Horizontal, symbol Device:R
- added R14: 150k, symbol Device:R
- added R15: 4.7k, Resistor_THT:R_Axial_DIN0207_L6.3mm_D2.5mm_P7.62mm_Horizontal, symbol Device:R
- added SW1: DPDT push-pull RV1, symbol Switch:SW_DPDT_x2
- C1: value 100p -> 47p
- J1: value IN (from PASSIVE jack NC lug) -> IN (от SW1B, экранир. провод)
- J3: value ACTIVE jack Tip/Sleeve -> OUT (к SW1A) / GND
- RV1: value A25k VOLUME -> B500K push-pull (Musiclily M908) VOLUME; footprint Connector_Wire:SolderWire-0.5sqmm_1x03_P4.6mm_D0.9mm_OD2.1mm -> (none)
- U1: value MCP6022 -> MCP6022/OPA2316
Connections:
- net BAT+: now also J6.1 (Pin_1)
- net GND: now also D1.1 (K), J4.S, J5.2 (Pin_2), J7.2 (Pin_2), R13.2, SW1.6 (C)
- net IN: now also SW1.5 (B)
- net OUT: now also R13.1, SW1.1 (A)
- net VCC: now also R15.1
- net at RV1.2: now also C13.2, R14.2, SW1.3 (C), SW1.4 (A); no longer R9.1
- net at RV1.3: now also C13.1, J5.1 (Pin_1), R14.1; no longer C9.2
- new net: C9.2, R9.1
- new net: J4.T, SW1.2 (B)
- new net BAT-: J4.R, J6.2 (Pin_2)
- new net LEDA: D1.2 (A), J7.1 (Pin_1), R15.2
Other:
- note added: "J1: экранированный провод от SW1B (жила=IN, оплётка=GND). J2: OUT+ модуля TP4056 с защитой (DW01) J3: OUT -> SW1A, GND -> Sleeve выходного джека. RV2/RV3: потенциометры BASS/TREBLE, вывод 3 = по часовой C2, C4-C7: плёночные (MKT/MKP), C1, C8: керамика C0G/NP0, C3/C9: электролит 10-16 В, C10/C12: 100 мкФ 10 В"
- note added: "SW1 — DPDT-переключатель потенциометра RV1 (push-pull Musiclily M908): НАЖАТ = АКТИВ: 2-1 (выход платы -> Tip), 5-4 (громкость -> вход платы) ВЫТЯНУТ = ПАССИВ: 2-3 (громкость -> Tip напрямую), 5-6 (вход платы -> земля) Какие крайние лепестки замкнуты в каком положении — проверить тестером (если наоборот — просто поменять местами провода на крайних лепестках). Питание: моно-штекер замыкает Ring-Sl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"
- note added: "ВНЕ ПЛАТЫ (на корпусе гитары)"
- note added: "ВЫХОД (громкость теперь до буфера, RV1)"
- note removed: "J1: экранированный провод от NC-лепестка ПАССИВНОГО джека (жила=IN, оплётка=GND) J2: OUT+ модуля TP4056 с защитой (DW01). OUT− модуля — сразу на кольцо (Ring) АКТИВНОГО джека J3: АКТИВНЫЙ стерео-джек TRS: T=OUT, S=GND. Моно-штекер замыкает R на S и включает питание RV1-RV3: потенциометры на корпусе гитары, вывод 3 = крайний по часовой стрелке C2, C4-C7: плёночные (MKT/MKP), C1, C8: керамика C0G/N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"
- note removed: "ГРОМКОСТЬ И ВЫХОД"
- moved on the sheet: R9, RV1

Commit message: понятнее для меня подключение jeck
Parts:
- J4: value Выход 6.3 стерео TRS -> Выход 6.3 Mono
- RV1: value B500K push-pull (Musiclily M908) VOLUME -> B500K push-pull VOLUME
Connections:
- net BAT+: now also SW1.1 (A), SW1.2 (B)
- net GND: now also J6.2 (Pin_2)
- net IN: no longer SW1.5 (B)
- net LEDA: no longer D1.2 (A), R15.2
- net OUT: no longer SW1.1 (A)
- net at C13.2, R14.2, RV1.2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: now also J4.T; no longer SW1.3 (C)
- net BAT-: no longer names the net of J4.R
- net BAT-: no longer J6.2 (Pin_2)
- new net: D1.2 (A), R15.2
- new net In: SW1.5 (B)
Other:
- note added: "ВЫХОД"
- note removed: "ВЫХОД (громкость теперь до буфера, RV1)"
- moved on the sheet: C1, C10, C11, C12, C13, C2, C3, C4, C5, C6, C7, C8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

Commit message: мой вариант
Connections:
- net In is gone; now on an unnamed net: SW1.5 (B)
- net BAT+: no longer J6.1 (Pin_1), SW1.1 (A)
- net GND: now also J4.R; no longer SW1.6 (C)
- net IN: now also SW1.6 (C)
- net at C13.2, R14.2, RV1.2: no longer J4.T, SW1.4 (A)
- net BAT IN+: now reaches SW1.3 (C)
- net BAT IN+: now also J6.1 (Pin_1)
- new net: J4.T, SW1.4 (A)
Other:
- moved on the sheet: C13, J4, J5, J6, R14, RV1, SW1A, SW1B

Commit message: кутерьма с коннекторами
Connections:
- net BAT IN+: now also J3.1 (Pin_1)
- net BAT+: no longer J2.1 (Pin_1)
- net GND: now also SW1.1 (A)
- net OUT: no longer J3.1 (Pin_1)
- new net BAT +: J2.1 (Pin_1)
Other:
- moved on the sheet: J1, J2, J3, J6, J7, SW1A

Commit message: переделка входного каскада
Parts:
- J4: value Выход 6.3 Mono -> Гнездо 6.3 стерео TRS
Connections:
- net BAT + is gone; now on net BAT+: J2.1 (Pin_1)
- net BAT+: now also J6.1 (Pin_1); no longer SW1.2 (B)
- net GND: no longer J4.R, J6.2 (Pin_2), SW1.1 (A)
- net LEDA: now also D1.2 (A), R15.2
- net OUT: now also J3.1 (Pin_1), SW1.3 (C)
- net TIP: now reaches J4.T, SW1.4 (A)
- net TIP: now also SW1.2 (B)
- removed net BAT IN+: J3.1 (Pin_1), J6.1 (Pin_1), SW1.3 (C)
- new net BAT-: J4.R, J6.2 (Pin_2)
- no-connect marks 0 -> 1
Other:
- note added: "SW1 — DPDT-переключатель потенциометра RV1 (push-pull Musiclily M908): АКТИВ: 5-6 (громкость -> вход платы IN), 2-3 (выход платы OUT -> Tip) ПАССИВ: 5-4 (громкость -> Tip напрямую), 2-1 (свободен: выход платы отключён) Какое положение ручки какое — проверить тестером (при необходимости поменять местами провода на крайних лепестках ОБЕИХ секций). Питание: J4 — стерео-гнездо TRS, кабель обычный мон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"
- note removed: "SW1 — DPDT-переключатель потенциометра RV1 (push-pull Musiclily M908): НАЖАТ = АКТИВ: 2-1 (выход платы -> Tip), 5-4 (громкость -> вход платы) ВЫТЯНУТ = ПАССИВ: 2-3 (громкость -> Tip напрямую), 5-6 (вход платы -> земля) Какие крайние лепестки замкнуты в каком положении — проверить тестером (если наоборот — просто поменять местами провода на крайних лепестках). Питание: моно-штекер замыкает Ring-Sl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"
- moved on the sheet: C1, C2, C3, C4, C5, C6, C7, C8, C9, J1, J2, J3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
